File: vstupy.sch (EAGLE design)
At the start: 43 parts, among them IC1 4012N, IC2 4012N, IC3 4075N

Commit message: uprava desky
Parts:
- removed IC1, IC2: 4012N, 40xx:4012N
- removed IC3: 4075N, 40xx:4075N
- removed SL1: (no value), con-amp-quick:M12
- added OK4, OK5: PC847, optocoupler:PC847
- added R25, R26, R27, R28, R29, R30, R31, R32, R33, R34, R35, R36, R37, R38, R39, R40: (no value), resistor:R-EU_0204/5
- added U$1: PRO-MINI, Arduino-clone:PRO-MINI
- added WEMOS1: (no value), esp8266modules:WEMOS-D1-MINI
- added X13, X14, X15, X16, X17, X18, X19, X20: (no value), con-wago-508:W237-3E
Connections:
- removed net +5V: R13.1, R14.1, R15.1, R16.1, R17.1, R18.1, R19.1, R20.1, R21.1, R22.1, R23.1, R24.1
- removed net N$10 (its old number): OK3B.A, R10.2
- removed net N$11 (its old number): OK3C.A, R11.2
- removed net N$12 (its old number): OK3D.A, R12.2
- removed net N$46: IC2A.I0, OK3A.COL, R21.2, SL1.9
- removed net N$9 (its old number): OK3A.A, R9.2
- new net +3V3: R10.1, R11.1, R12.1, R13.1, R14.1, R15.1, R16.1, R21.1, R22.1, R23.1, R24.1, R29.1, R30.1, R31.1, R32.1, R37.1, R38.1, R39.1, R40.1, R9.1
- new net N$17: OK2A.COL, R9.2, U$1.D2
- new net N$18: OK2B.COL, R10.2, U$1.D3
- new net N$19: OK2C.COL, R11.2, U$1.D4
- new net N$20: OK2D.COL, R12.2, U$1.D5
- new net N$31: OK1A.COL, R13.2, U$1.D6
- new net N$32: OK1B.COL, R14.2, U$1.D7
- new net N$33: OK3C.COL, R23.2, U$1.A2
- new net N$34: OK1C.COL, R15.2, U$1.D8
- new net N$35: OK1D.COL, R16.2, U$1.D9
- new net N$36: OK3D.COL, R24.2, U$1.A3
- new net N$37: OK4A.A, R25.2
- new net N$51: OK5C.A, R35.2
- new net N$52: OK5D.A, R36.2
- new net N$53: R33.1, X17-1.KL
- new net N$54: R34.1, X18-1.KL
- new net N$55: R35.1, X19-1.KL
- new net N$56: R36.1, X20-1.KL
- new net N$57: OK5A.COL, R37.2, U$1.A4
- new net N$58: OK5B.COL, R38.2, U$1.A5
- new net N$59: OK5C.COL, R39.2, U$1.A6
- new net N$60: OK5D.COL, R40.2, U$1.A7
- new net N$61: OK4B.COL, R30.2, U$1.D11
- net +12V: now also X13-2.KL, X14-2.KL, X15-2.KL, X16-2.KL, X17-2.KL, X18-2.KL, X19-2.KL, X20-2.KL
- net GND: now also OK2A.EMIT, OK4A.C, OK4A.EMIT, OK4B.C, OK4B.EMIT, OK4C.C, OK4C.EMIT, OK4D.C, OK4D.EMIT, OK5A.C, OK5A.EMIT, OK5B.C, OK5B.EMIT, OK5C.C, OK5C.EMIT, OK5D.C, OK5D.EMIT, X13-3.KL, X14-3.KL, X15-3.KL, X16-3.KL, X17-3.KL, X18-3.KL, X19-3.KL, X20-3.KL
- net N$21: now also OK3A.A, R17.2; no longer R9.1, X9-1.KL
- net N$22: now also OK3B.A, R18.2; no longer R10.1, X10-1.KL
- net N$23: now also OK3C.A, R19.2; no longer R11.1, X11-1.KL
- net N$24: now also OK3D.A, R20.2; no longer R12.1, X12-1.KL
- net N$25: now also R17.1, X9-1.KL; no longer IC1A.O, IC3A.I0, IC3A.I1, IC3A.I2
- net N$26: now also R18.1, X10-1.KL; no longer IC1B.O, IC3B.I0, IC3B.I1, IC3B.I2
- net N$27: now also R19.1, X11-1.KL; no longer IC2A.O, IC3C.I0, IC3C.I1, IC3C.I2
- net N$28: now also R20.1, X12-1.KL; no longer IC2B.I0, IC3A.O
- net N$29: now also OK3A.COL, R21.2, U$1.A0; no longer IC2B.I1, IC3B.O
- net N$30: now also OK3B.COL, R22.2, U$1.A1; no longer IC2B.I2, IC2B.I3, IC3C.O
- net N$38: now also OK4B.A, R26.2; no longer IC1A.I0, OK1A.COL, R13.2, SL1.1
- net N$39: now also OK4C.A, R27.2; no longer IC1A.I1, OK1B.COL, R14.2, SL1.2
- net N$40: now also OK4D.A, R28.2; no longer IC1A.I2, OK1C.COL, R15.2, SL1.3
- net N$41: now also R25.1, X13-1.KL; no longer IC1A.I3, OK1D.COL, R16.2, SL1.4
- net N$42: now also R26.1, X14-1.KL; no longer IC1B.I0, OK2A.COL, R17.2, SL1.5
- net N$43: now also R27.1, X15-1.KL; no longer IC1B.I1, OK2B.COL, R18.2, SL1.6
- net N$44: now also R28.1, X16-1.KL; no longer IC1B.I2, OK2C.COL, R19.2, SL1.7
- net N$45: now also OK4A.COL, R29.2, U$1.D10; no longer IC1B.I3, OK2D.COL, R20.2, SL1.8
- net N$47: now also OK4C.COL, R31.2, U$1.D12; no longer IC2A.I1, OK3B.COL, R22.2, SL1.10
- net N$48: now also OK4D.COL, R32.2, U$1.D13; no longer IC2A.I2, OK3C.COL, R23.2, SL1.11
- net N$49: now also OK5A.A, R33.2; no longer IC2A.I3, OK3D.COL, R24.2, SL1.12
- net N$50: now also OK5B.A, R34.2; no longer OK2A.EMIT
Other:
- moved on the sheet: OK2A, OK2B, OK2C, OK2D, OK3A, OK3B, OK3C, OK3D, R10, R11, R12, R17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

Commit message: +
Parts:
- added SL1: (no value), con-amp-quick:M04
Connections:
- new net N$46: SL1.1, U$1.TX0, WEMOS1.RX
- new net N$62: SL1.2, U$1.RX1, WEMOS1.TX
- net +3V3: now also SL1.3, U$1.RAW, WEMOS1.3V3, WEMOS1.RESET
- net GND: now also SL1.4, U$1.GND, WEMOS1.GND
Changed lines of the file:
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@@
 <part name="U$1" library="Arduino-clone" deviceset="PRO-MINI" device=""/>
 <part name="WEMOS1" library="esp8266modules" deviceset="WEMOS-D1-MINI" device=""/>
+<part name="GND21" library="supply1" deviceset="GND" device=""/>
+<part name="GND22" library="supply1" deviceset="GND" device=""/>
+<part name="+3V2" library="supply1" deviceset="+3V3" device=""/>
+<part name="SL1" library="con-amp-quick" deviceset="M04" device=""/>
+<part name="GND23" library="supply1" deviceset="GND" device=""/>
+<part name="+3V3" library="supply1" deviceset="+3V3" device=""/>
 </parts>
 <sheets>
@@
 <instance part="U$1" gate="G$1" x="96.52" y="12.7"/>
 <instance part="WEMOS1" gate="D1" x="111.76" y="-60.96"/>
+<instance part="GND21" gate="1" x="129.54" y="27.94"/>
+<instance part="GND22" gate="1" x="139.7" y="-68.58"/>
+<instance part="+3V2" gate="G$1" x="93.98" y="-71.12" rot="R180"/>
+<instance part="SL1" gate="G$1" x="165.1" y="-60.96" rot="R180"/>
+<instance part="GND23" gate="1" x="160.02" y="-68.58"/>
+<instance part="+3V3" gate="G$1" x="157.48" y="-63.5" rot="R90"/>
 </instances>
 <busses>
@@
 <wire x1="2.54" y1="-279.4" x2="20.32" y2="-279.4" width="0.1524" layer="91"/>
 <wire x1="20.32" y1="-279.4" x2="20.32" y2="-274.32" width="0.1524" layer="91"/>
+</segment>
+<segment>
+<pinref part="GND21" gate="1" pin="GND"/>
+<pinref part="U$1" gate="G$1" pin="GND"/>
+<wire x1="129.54" y1="30.48" x2="114.3" y2="30.48" width="0.1524" layer="91"/>
+</segment>
+<segment>
+<pinref part="WEMOS1" gate="D1" pin="GND"/>
+<pinref part="GND22" gate="1" pin="GND"/>
+<wire x1="129.54" y1="-66.04" x2="139.7" y2="-66.04" width="0.1524" layer="91"/>
+</segment>
+<segment>
+<pinref part="SL1" gate="G$1" pin="4"/>
+<pinref part="GND23" gate="1" pin="GND"/>
 </segment>
 </net>
@@
 <wire x1="30.48" y1="45.72" x2="30.48" y2="20.32" width="0.1524" layer="91"/>
 <junction x="30.48" y="45.72"/>
+<wire x1="30.48" y1="99.06" x2="121.92" y2="99.06" width="0.1524" layer="91"/>
+<wire x1="121.92" y1="99.06" x2="121.92" y2="33.02" width="0.1524" layer="91"/>
+<pinref part="U$1" gate="G$1" pin="RAW"/>
+<wire x1="121.92" y1="33.02" x2="114.3" y2="33.02" width="0.1524" layer="91"/>
+</segment>
+<segment>
+<pinref part="WEMOS1" gate="D1" pin="3V3"/>
+<pinref part="+3V2" gate="G$1" pin="+3V3"/>
+<pinref part="WEMOS1" gate="D1" pin="RESET"/>
+<wire x1="96.52" y1="-50.8" x2="93.98" y2="-50.8" width="0.1524" layer="91"/>
+<wire x1="93.98" y1="-50.8" x2="93.98" y2="-68.58" width="0.1524" layer="91"/>
+<junction x="93.98" y="-68.58"/>
+<wire x1="93.98" y1="-68.58" x2="96.52" y2="-68.58" width="0.1524" layer="91"/>
+</segment>
+<segment>
+<pinref part="SL1" gate="G$1" pin="3"/>
+<pinref part="+3V3" gate="G$1" pin="+3V3"/>
 </segment>
 </net>
@@
 </segment>
 </net>
+<net name="N$46" class="0">
+<segment>
+<pinref part="U$1" gate="G$1" pin="TX0"/>
+<wire x1="73.66" y1="33.02" x2="68.58" y2="33.02" width="0.1524" layer="91"/>
+<wire x1="68.58" y1="33.02" x2="68.58" y2="55.88" width="0.1524" layer="91"/>
+<wire x1="68.58" y1="55.88" x2="152.4" y2="55.88" width="0.1524" layer="91"/>
+<wire x1="152.4" y1="55.88" x2="152.4" y2="-53.34" width="0.1524" layer="91"/>
+<pinref part="WEMOS1" gate="D1" pin="RX"/>
+<wire x1="152.4" y1="-53.34" x2="129.54" y2="-53.34" width="0.1524" layer="91"/>
+<pinref part="SL1" gate="G$1" pin="1"/>
+<wire x1="160.02" y1="-58.42" x2="152.4" y2="-58.42" width="0.1524" layer="91"/>
+<wire x1="152.4" y1="-58.42" x2="152.4" y2="-53.34" width="0.1524" layer="91"/>
+<junction x="152.4" y="-53.34"/>
+</segment>
+</net>
+<net name="N$62" class="0">
+<segment>
+<pinref part="U$1" gate="G$1" pin="RX1"/>
+<wire x1="73.66" y1="30.48" x2="71.12" y2="30.48" width="0.1524" layer="91"/>
+<wire x1="71.12" y1="30.48" x2="71.12" y2="53.34" width="0.1524" layer="91"/>
+<wire x1="71.12" y1="53.34" x2="149.86" y2="53.34" width="0.1524" layer="91"/>
+<wire x1="149.86" y1="53.34" x2="149.86" y2="-48.26" width="0.1524" layer="91"/>
+<pinref part="WEMOS1" gate="D1" pin="TX"/>
+<wire x1="149.86" y1="-48.26" x2="129.54" y2="-48.26" width="0.1524" layer="91"/>
+<wire x1="129.54" y1="-48.26" x2="129.54" y2="-50.8" width="0.1524" layer="91"/>
+<pinref part="SL1" gate="G$1" pin="2"/>
+<wire x1="160.02" y1="-60.96" x2="149.86" y2="-60.96" width="0.1524" layer="91"/>
+<wire x1="149.86" y1="-60.96" x2="149.86" y2="-48.26" width="0.1524" layer="91"/>
+<junction x="149.86" y="-48.26"/>
+</segment>
+</net>

Commit message: uprava desky
Parts:
- removed OK4, OK5: PC847, optocoupler:PC847
- removed R17, R18, R19, R20, R21, R22, R23, R24, R33, R34, R35, R36, R37, R38, R39, R40: (no value), resistor:R-EU_0204/5
- removed SL1: (no value), con-amp-quick:M04
- removed WEMOS1: (no value), esp8266modules:WEMOS-D1-MINI
- removed X10, X11, X12, X17, X18, X19, X20: (no value), con-wago-508:W237-3E
Connections:
- removed net +3V3: R10.1, R11.1, R12.1, R13.1, R14.1, R15.1, R16.1, R21.1, R22.1, R23.1, R24.1, R29.1, R30.1, R31.1, R32.1, R37.1, R38.1, R39.1, R40.1, R9.1, SL1.3, U$1.RAW, WEMOS1.3V3, WEMOS1.RESET
- removed net N$24: OK3D.A, R20.2
- removed net N$25: R17.1, X9-1.KL
- removed net N$26: R18.1, X10-1.KL
- removed net N$27: R19.1, X11-1.KL
- removed net N$28: R20.1, X12-1.KL
- removed net N$29: OK3A.COL, R21.2, U$1.A0
- removed net N$30: OK3B.COL, R22.2, U$1.A1
- removed net N$31: OK1A.COL, R13.2, U$1.D6
- removed net N$32: OK1B.COL, R14.2, U$1.D7
- removed net N$33: OK3C.COL, R23.2, U$1.A2
- removed net N$34: OK1C.COL, R15.2, U$1.D8
- removed net N$36: OK3D.COL, R24.2, U$1.A3
- removed net N$46: SL1.1, U$1.TX0, WEMOS1.RX
- removed net N$49: OK5A.A, R33.2
- removed net N$50: OK5B.A, R34.2
- removed net N$51: OK5C.A, R35.2
- removed net N$52: OK5D.A, R36.2
- removed net N$53: R33.1, X17-1.KL
- removed net N$54: R34.1, X18-1.KL
- removed net N$55: R35.1, X19-1.KL
- removed net N$56: R36.1, X20-1.KL
- removed net N$57: OK5A.COL, R37.2, U$1.A4
- removed net N$58: OK5B.COL, R38.2, U$1.A5
- removed net N$59: OK5C.COL, R39.2, U$1.A6
- removed net N$60: OK5D.COL, R40.2, U$1.A7
- removed net N$62: SL1.2, U$1.RX1, WEMOS1.TX
- new net +5V: R10.1, R11.1, R12.1, R13.1, R14.1, R15.1, R16.1, R29.1, R30.1, R31.1, R32.1, R9.1, U$1.RAW, X9-2.KL
- net +12V: now also X9-1.KL; no longer X10-2.KL, X11-2.KL, X12-2.KL, X17-2.KL, X18-2.KL, X19-2.KL, X20-2.KL, X9-2.KL
- net GND: no longer OK4A.C, OK4A.EMIT, OK4B.C, OK4B.EMIT, OK4C.C, OK4C.EMIT, OK4D.C, OK4D.EMIT, OK5A.C, OK5A.EMIT, OK5B.C, OK5B.EMIT, OK5C.C, OK5C.EMIT, OK5D.C, OK5D.EMIT, SL1.4, WEMOS1.GND, X10-3.KL, X11-3.KL, X12-3.KL, X17-3.KL, X18-3.KL, X19-3.KL, X20-3.KL
- net N$17: now also U$1.D5; no longer U$1.D2
- net N$18: now also U$1.D4; no longer U$1.D3
- net N$19: now also U$1.D3; no longer U$1.D4
- net N$20: now also U$1.D2; no longer U$1.D5
- net N$21: now also OK1A.COL, R13.2, U$1.D9; no longer OK3A.A, R17.2
- net N$22: now also OK1B.COL, R14.2, U$1.D8; no longer OK3B.A, R18.2
- net N$23: now also OK1C.COL, R15.2, U$1.D7; no longer OK3C.A, R19.2
- net N$35: now also U$1.D6; no longer U$1.D9
- net N$37: now also OK3A.A; no longer OK4A.A
- net N$38: now also OK3B.A; no longer OK4B.A
- net N$39: now also OK3C.A; no longer OK4C.A
- net N$40: now also OK3D.A; no longer OK4D.A
- net N$45: now also OK3A.COL, U$1.D13; no longer OK4A.COL, U$1.D10
- net N$47: now also OK3C.COL, U$1.D11; no longer OK4C.COL, U$1.D12
- net N$48: now also OK3D.COL, U$1.D10; no longer OK4D.COL, U$1.D13
- net N$61: now also OK3B.COL, U$1.D12; no longer OK4B.COL, U$1.D11
Other:
- moved on the sheet: OK3A, OK3B, OK3C, OK3D, R25, R26, R27, R28, R29, R30, R31, R32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
